File: power_share.kicad_pcb (KiCad board)
At the start: 2 copper layers, 32.5 x 21.1 mm, 14 parts, among them J1 Conn_01x02, J2 Conn_01x03, Q1 NX3008NBKW, Q2 NX3008NBKW, U1 LTC4370

Commit message: Added logo
Parts:
- added G***: LOGO, Logos:asian_tiger, F.Cu at (130.6, 93.5)
- added G***: LOGO, Logos:asian_tiger, F.Cu at (129.8, 90.2)
- added G***: LOGO, Logos:asian_tiger, F.Cu at (125.0, 90.2)
- added G***: LOGO, Logos:asian_tiger, F.Cu at (127.3, 88.1)
- added G***: LOGO, Logos:asian_tiger, F.Cu at (121.4, 87.4)
- added G***: LOGO, Logos:asian_tiger, F.Cu at (129.3, 94.5)
- added G***: LOGO, Logos:asian_tiger, F.Cu at (126.7, 92.2)
- added G***: LOGO, Logos:asian_tiger, F.Cu at (127.8, 92.5)
Other:
- board text added: "Current Balancer v0.1 Hyiger Designs"
- board text removed: "Current Balancer"
