File: power_share.sch (KiCad schematic (older format))
At the start: 14 parts, among them J1 Conn_01x02, J2 Conn_01x03, Q1 NX3008NBKW, Q2 NX3008NBKW, U1 LTC4370

Commit message: cleaned up layout
Parts:
- Q1, Q2: symbol Transistor_FET:NX3008NBKW -> power_share-rescue:NX3008NBKW-Transistor_FET
- U1: symbol Power_Management:LTC4370 -> power_share-rescue:LTC4370-Power_Management
Connections:
- wire segments 50 -> 49
Changed lines of the file:
@@
 $EndDescr
 $Comp
-L Transistor_FET:NX3008NBKW Q1
+L power_share-rescue:NX3008NBKW-Transistor_FET Q1
 U 1 1 5D158ED3
 P 5770 2670
@@
 $EndComp
 $Comp
-L Transistor_FET:NX3008NBKW Q2
+L power_share-rescue:NX3008NBKW-Transistor_FET Q2
 U 1 1 5D1599E4
 P 5770 4360
@@
 U 1 1 5D1689F8
 P 5370 4165
-F 0 "C4" H 5462 4211 50  0000 L CNN
-F 1 "39nF" H 5462 4120 50  0000 L CNN
+F 0 "C4" H 5185 4135 50  0000 L CNN
+F 1 "39nF" H 5125 4215 50  0000 L CNN
 F 2 "Capacitor_SMD:C_0603_1608Metric_Pad1.05x0.95mm_HandSolder" H 5370 4165 50  0001 C CNN
 F 3 "~" H 5370 4165 50  0001 C CNN
@@
 L power:GND #PWR01
 U 1 1 5D17B2A4
-P 4620 3570
-F 0 "#PWR01" H 4620 3320 50  0001 C CNN
-F 1 "GND" H 4625 3397 50  0000 C CNN
-F 2 "" H 4620 3570 50  0001 C CNN
-F 3 "" H 4620 3570 50  0001 C CNN
-	1    4620 3570
+P 4620 3620
+F 0 "#PWR01" H 4620 3370 50  0001 C CNN
+F 1 "GND" H 4625 3447 50  0000 C CNN
+F 2 "" H 4620 3620 50  0001 C CNN
+F 3 "" H 4620 3620 50  0001 C CNN
+	1    4620 3620
 	1    0    0    -1
 $EndComp
 Wire Wire Line
 	4870 3665 4755 3665
-Wire Wire Line
-	4620 3570 4620 3575
-Wire Wire Line
-	4620 3545 4620 3570
-Connection ~ 4620 3570
 $Comp
 L Device:C_Small C2
@@
 P 4620 3470
 F 0 "C2" H 4712 3516 50  0000 L CNN
-F 1 "100nF" H 4712 3425 50  0000 L CNN
+F 1 "100nF" H 4360 3390 50  0000 L CNN
 F 2 "Capacitor_SMD:C_0603_1608Metric_Pad1.05x0.95mm_HandSolder" H 4620 3470 50  0001 C CNN
 F 3 "~" H 4620 3470 50  0001 C CNN
@@
 P 4755 3765
 F 0 "R4" H 4814 3811 50  0000 L CNN
-F 1 "30.1k" H 4814 3720 50  0000 L CNN
+F 1 "30.1k" H 4515 3690 50  0000 L CNN
 F 2 "Resistor_SMD:R_0603_1608Metric_Pad1.05x0.95mm_HandSolder" H 4755 3765 50  0001 C CNN
 F 3 "~" H 4755 3765 50  0001 C CNN
@@
 Wire Wire Line
 	4870 3515 4760 3515
-Wire Wire Line
-	4760 3515 4755 3570
-Wire Wire Line
-	4755 3570 4620 3570
 Wire Wire Line
 	4870 3815 4870 3865
@@
 	7320 3430 7445 3430
 $Comp
-L Power_Management:LTC4370 U1
+L power_share-rescue:LTC4370-Power_Management U1
 U 1 1 5D15CEC4
 P 5570 3515
@@
 	1    0    0    -1
 $EndComp
+Wire Wire Line
+	4760 3515 4760 3570
+Wire Wire Line
+	4760 3570 4620 3570
+Wire Wire Line
+	4620 3620 4620 3570
+Connection ~ 4620 3570
 $EndSCHEMATC
